Commit message: imu-ros2 bridge, imu_opp, navigation configuration setup

File: ros2_ws/src/wheelchair_description/urdf/wheelchair.urdf.xacro (robot description, xacro)
@@ -1,19 +1,15 @@
 <?xml version="1.0"?>
 <robot xmlns:xacro="http://www.ros.org/wiki/xacro" name="wheelchair">
-  <!-- Args (override via launch/yaml) -->
-  <xacro:arg name="base_length" default="0.50"/>    <!-- Chassis length (x)-->
-  <xacro:arg name="base_width"  default="0.50"/>    <!-- Chassis width (y)-->
-  <xacro:arg name="base_height" default="0.50"/>    <!-- Chassis thickness (z)-->
-  <!-- base_link pose relative to base_footprint (ground frame) -->
-  <xacro:arg name="base_z" default="0.0"/>    <!-- base_footprint -> base_link z offset -->
-  <!-- RealSense root frame mount: camera_link -->
-  <!-- Camera mount pose relative to base_link -->
-  <xacro:arg name="camera_x" default="0.30"/>   <!-- Forward-Backward (x)-->
-  <xacro:arg name="camera_y" default="0.0"/>    <!-- Left-Right (y)-->
-  <xacro:arg name="camera_z" default="0.60"/>   <!-- Up-Down (z)-->
-  <xacro:arg name="camera_roll"  default="0.0"/>    <!-- in rad-->
-  <xacro:arg name="camera_pitch" default="0.0"/>    <!-- in rad-->
-  <xacro:arg name="camera_yaw"   default="0.0"/>    <!-- in rad-->
-  <!-- LiDAR mount -->
+  <!-- Args -->
+  <xacro:arg name="base_length" default="0.50"/>
+  <xacro:arg name="base_width"  default="0.50"/>
+  <xacro:arg name="base_height" default="0.50"/>
+  <xacro:arg name="base_z" default="0.0"/>
+  <xacro:arg name="camera_x" default="0.30"/>
+  <xacro:arg name="camera_y" default="0.0"/>
+  <xacro:arg name="camera_z" default="0.60"/>
+  <xacro:arg name="camera_roll"  default="0.0"/>
+  <xacro:arg name="camera_pitch" default="0.0"/>
+  <xacro:arg name="camera_yaw"   default="0.0"/>
   <xacro:arg name="lidar_x" default="0.25"/>
   <xacro:arg name="lidar_y" default="0.0"/>
@@ -22,5 +18,4 @@
   <xacro:arg name="lidar_pitch" default="0.0"/>
   <xacro:arg name="lidar_yaw"   default="0.0"/>
-  <!-- IMU mount -->
   <xacro:arg name="imu_x" default="0.00"/>
   <xacro:arg name="imu_y" default="0.0"/>
@@ -29,36 +24,50 @@
   <xacro:arg name="imu_pitch" default="0.0"/>
   <xacro:arg name="imu_yaw"   default="0.0"/>
+  <!-- Properties from args -->
+  <xacro:property name="base_length_v" value="$(arg base_length)"/>
+  <xacro:property name="base_width_v"  value="$(arg base_width)"/>
+  <xacro:property name="base_height_v" value="$(arg base_height)"/>
+  <xacro:property name="base_z_v"      value="$(arg base_z)"/>
+  <xacro:property name="camera_x_v" value="$(arg camera_x)"/>
+  <xacro:property name="camera_y_v" value="$(arg camera_y)"/>
+  <xacro:property name="camera_z_v" value="$(arg camera_z)"/>
+  <xacro:property name="camera_roll_v"  value="$(arg camera_roll)"/>
+  <xacro:property name="camera_pitch_v" value="$(arg camera_pitch)"/>
+  <xacro:property name="camera_yaw_v"   value="$(arg camera_yaw)"/>
+  <xacro:property name="lidar_x_v" value="$(arg lidar_x)"/>
+  <xacro:property name="lidar_y_v" value="$(arg lidar_y)"/>
+  <xacro:property name="lidar_z_v" value="$(arg lidar_z)"/>
+  <xacro:property name="lidar_roll_v"  value="$(arg lidar_roll)"/>
+  <xacro:property name="lidar_pitch_v" value="$(arg lidar_pitch)"/>
+  <xacro:property name="lidar_yaw_v"   value="$(arg lidar_yaw)"/>
+  <xacro:property name="imu_x_v" value="$(arg imu_x)"/>
+  <xacro:property name="imu_y_v" value="$(arg imu_y)"/>
+  <xacro:property name="imu_z_v" value="$(arg imu_z)"/>
+  <xacro:property name="imu_roll_v"  value="$(arg imu_roll)"/>
+  <xacro:property name="imu_pitch_v" value="$(arg imu_pitch)"/>
+  <xacro:property name="imu_yaw_v"   value="$(arg imu_yaw)"/>
   <material name="gray"><color rgba="0.6 0.6 0.6 1"/></material>
   <material name="black"><color rgba="0.1 0.1 0.1 1"/></material>
-  <!-- base_footprint: ground-projected frame for navigation (z=0) -->
-  <link name="base_footprint"/>   <!-- Ground reference frame -->
-  <!-- base_link: robot body frame -->
-  <!-- Main body frame -->
+  <link name="base_footprint"/>
   <link name="base_link">
-    <visual>    <!-- RViz visual geometry -->
-      <origin xyz="0 0 ${float(arg('base_height'))/2.0}" rpy="0 0 0"/>
-      <geometry>    <!-- Visual shape -->
-        <box size="${arg('base_length')} ${arg('base_width')} ${arg('base_height')}"/>
+    <visual>
+      <origin xyz="0 0 ${float(base_height_v)/2.0}" rpy="0 0 0"/>
+      <geometry>
+        <box size="${base_length_v} ${base_width_v} ${base_height_v}"/>
       </geometry>
       <material name="gray"/>
     </visual>
-    <collision>   <!-- Collision geometry (planning/sim) -->
-      <origin xyz="0 0 ${float(arg('base_height'))/2.0}" rpy="0 0 0"/>
-      <geometry>    <!-- Collision shape -->
-        <box size="${arg('base_length')} ${arg('base_width')} ${arg('base_height')}"/>
+    <collision>
+      <origin xyz="0 0 ${float(base_height_v)/2.0}" rpy="0 0 0"/>
+      <geometry>
+        <box size="${base_length_v} ${base_width_v} ${base_height_v}"/>
       </geometry>
     </collision>
   </link>
-  <!-- base_footprint -> base_link -->
-  <!-- Fixed transform from ground frame to body frame -->
-  <joint name="base_joint" type="fixed">    <!-- Rigid connection (no motion) -->
+  <joint name="base_joint" type="fixed">
     <parent link="base_footprint"/>
     <child link="base_link"/>
-    <origin xyz="0 0 ${arg('base_z')}" rpy="0 0 0"/>
+    <origin xyz="0 0 ${base_z_v}" rpy="0 0 0"/>
   </joint>
-  <!-- RealSense root frame: camera_link
-       RealSense topics use frame_id like camera_color_optical_frame.
-       realsense-ros typically publishes TF camera_link -> ... -> camera_color_optical_frame.
-       So we only mount camera_link here to avoid TF conflicts. -->
   <link name="camera_link">
     <visual>
@@ -71,12 +80,10 @@
     <parent link="base_link"/>
     <child link="camera_link"/>
-    <origin xyz="${arg('camera_x')} ${arg('camera_y')} ${arg('camera_z')}"
-            rpy="${arg('camera_roll')} ${arg('camera_pitch')} ${arg('camera_yaw')}"/>
+    <origin xyz="${camera_x_v} ${camera_y_v} ${camera_z_v}"
+            rpy="${camera_roll_v} ${camera_pitch_v} ${camera_yaw_v}"/>
   </joint>
-  <!-- LiDAR base (mount point for driver-provided TF chain)-->
   <link name="ldlidar_base">
     <visual>
       <origin xyz="0 0 0" rpy="0 0 0"/>
-      <!-- Referenced LiDAR CAD Design-->
       <geometry><cylinder radius="0.027" length="0.0348"/></geometry>
       <material name="black"/>
@@ -86,8 +93,7 @@
     <parent link="base_link"/>
     <child link="ldlidar_base"/>
-    <origin xyz="${arg('lidar_x')} ${arg('lidar_y')} ${arg('lidar_z')}"
-            rpy="${arg('lidar_roll')} ${arg('lidar_pitch')} ${arg('lidar_yaw')}"/>
+    <origin xyz="${lidar_x_v} ${lidar_y_v} ${lidar_z_v}"
+            rpy="${lidar_roll_v} ${lidar_pitch_v} ${lidar_yaw_v}"/>
   </joint>
-  <!-- IMU -->
   <link name="imu_link">
     <visual>
@@ -100,6 +106,6 @@
     <parent link="base_link"/>
     <child link="imu_link"/>
-    <origin xyz="${arg('imu_x')} ${arg('imu_y')} ${arg('imu_z')}"
-            rpy="${arg('imu_roll')} ${arg('imu_pitch')} ${arg('imu_yaw')}"/>
+    <origin xyz="${imu_x_v} ${imu_y_v} ${imu_z_v}"
+            rpy="${imu_roll_v} ${imu_pitch_v} ${imu_yaw_v}"/>
   </joint>
 </robot>

Commit message: new urdf with casters

File: ros2_ws/src/wheelchair_description/urdf/wheelchair.urdf.xacro (robot description, xacro)
@@ -1,15 +1,13 @@
 <?xml version="1.0"?>
 <robot xmlns:xacro="http://www.ros.org/wiki/xacro" name="wheelchair">
-  <!-- Args -->
+  <!-- ========================================================= -->
+  <!-- Arguments                                                 -->
+  <!-- ========================================================= -->
+  <!-- Base body -->
   <xacro:arg name="base_length" default="0.50"/>
   <xacro:arg name="base_width"  default="0.50"/>
   <xacro:arg name="base_height" default="0.50"/>
-  <xacro:arg name="base_z" default="0.171"/>
-  <xacro:arg name="camera_x" default="0.0"/>
-  <xacro:arg name="camera_y" default="0.0"/>
-  <xacro:arg name="camera_z" default="0.0"/>
-  <xacro:arg name="camera_roll"  default="0.0"/>
-  <xacro:arg name="camera_pitch" default="0.0"/>
-  <xacro:arg name="camera_yaw"   default="0.0"/>
+  <xacro:arg name="base_z"      default="0.171"/>
+  <!-- LiDAR mount -->
   <xacro:arg name="lidar_x" default="0.0"/>
   <xacro:arg name="lidar_y" default="0.0"/>
@@ -18,4 +16,5 @@
   <xacro:arg name="lidar_pitch" default="0.0"/>
   <xacro:arg name="lidar_yaw"   default="0.0"/>
+  <!-- IMU mount -->
   <xacro:arg name="imu_x" default="0.0"/>
   <xacro:arg name="imu_y" default="0.0"/>
@@ -24,15 +23,17 @@
   <xacro:arg name="imu_pitch" default="0.0"/>
   <xacro:arg name="imu_yaw"   default="0.0"/>
-  <!-- Properties from args -->
+  <!-- Front caster wheels -->
+  <xacro:arg name="front_caster_x"      default="0.30"/>
+  <xacro:arg name="front_caster_y"      default="0.20"/>
+  <xacro:arg name="front_caster_z"      default="0.05"/>
+  <xacro:arg name="front_caster_radius" default="0.05"/>
+  <xacro:arg name="front_caster_width"  default="0.03"/>
+  <!-- ========================================================= -->
+  <!-- Properties                                                -->
+  <!-- ========================================================= -->
   <xacro:property name="base_length_v" value="$(arg base_length)"/>
   <xacro:property name="base_width_v"  value="$(arg base_width)"/>
   <xacro:property name="base_height_v" value="$(arg base_height)"/>
   <xacro:property name="base_z_v"      value="$(arg base_z)"/>
-  <xacro:property name="camera_x_v" value="$(arg camera_x)"/>
-  <xacro:property name="camera_y_v" value="$(arg camera_y)"/>
-  <xacro:property name="camera_z_v" value="$(arg camera_z)"/>
-  <xacro:property name="camera_roll_v"  value="$(arg camera_roll)"/>
-  <xacro:property name="camera_pitch_v" value="$(arg camera_pitch)"/>
-  <xacro:property name="camera_yaw_v"   value="$(arg camera_yaw)"/>
   <xacro:property name="lidar_x_v" value="$(arg lidar_x)"/>
   <xacro:property name="lidar_y_v" value="$(arg lidar_y)"/>
@@ -47,6 +48,21 @@
   <xacro:property name="imu_pitch_v" value="$(arg imu_pitch)"/>
   <xacro:property name="imu_yaw_v"   value="$(arg imu_yaw)"/>
-  <material name="gray"><color rgba="0.6 0.6 0.6 1"/></material>
-  <material name="black"><color rgba="0.1 0.1 0.1 1"/></material>
+  <xacro:property name="front_caster_x_v"      value="$(arg front_caster_x)"/>
+  <xacro:property name="front_caster_y_v"      value="$(arg front_caster_y)"/>
+  <xacro:property name="front_caster_z_v"      value="$(arg front_caster_z)"/>
+  <xacro:property name="front_caster_radius_v" value="$(arg front_caster_radius)"/>
+  <xacro:property name="front_caster_width_v"  value="$(arg front_caster_width)"/>
+  <!-- ========================================================= -->
+  <!-- Materials                                                 -->
+  <!-- ========================================================= -->
+  <material name="gray">
+    <color rgba="0.6 0.6 0.6 1"/>
+  </material>
+  <material name="black">
+    <color rgba="0.1 0.1 0.1 1"/>
+  </material>
+  <!-- ========================================================= -->
+  <!-- Base                                                      -->
+  <!-- ========================================================= -->
   <link name="base_footprint"/>
   <link name="base_link">
@@ -70,34 +86,31 @@
     <origin xyz="0 0 ${base_z_v}" rpy="0 0 0"/>
   </joint>
-  <link name="camera_link">
+  <!-- ========================================================= -->
+  <!-- LiDAR                                                     -->
+  <!-- ========================================================= -->
+  <link name="lidar_link">
     <visual>
       <origin xyz="0 0 0" rpy="0 0 0"/>
-      <geometry><box size="0.09 0.025 0.025"/></geometry>
+      <geometry>
+        <cylinder radius="0.027" length="0.0348"/>
+      </geometry>
       <material name="black"/>
     </visual>
   </link>
-  <joint name="camera_mount_joint" type="fixed">
+  <joint name="lidar_joint" type="fixed">
     <parent link="base_link"/>
-    <child link="camera_link"/>
-    <origin xyz="${camera_x_v} ${camera_y_v} ${camera_z_v}"
-            rpy="${camera_roll_v} ${camera_pitch_v} ${camera_yaw_v}"/>
-  </joint>
-  <link name="ldlidar_base">
-    <visual>
-      <origin xyz="0 0 0" rpy="0 0 0"/>
-      <geometry><cylinder radius="0.027" length="0.0348"/></geometry>
-      <material name="black"/>
-    </visual>
-  </link>
-  <joint name="lidar_base_joint" type="fixed">
-    <parent link="base_link"/>
-    <child link="ldlidar_base"/>
+    <child link="lidar_link"/>
     <origin xyz="${lidar_x_v} ${lidar_y_v} ${lidar_z_v}"
             rpy="${lidar_roll_v} ${lidar_pitch_v} ${lidar_yaw_v}"/>
   </joint>
+  <!-- ========================================================= -->
+  <!-- IMU                                                       -->
+  <!-- ========================================================= -->
   <link name="imu_link">
     <visual>
       <origin xyz="0 0 0" rpy="0 0 0"/>
-      <geometry><box size="0.03 0.02 0.01"/></geometry>
+      <geometry>
+        <box size="0.03 0.02 0.01"/>
+      </geometry>
       <material name="black"/>
     </visual>
@@ -109,3 +122,46 @@
             rpy="${imu_roll_v} ${imu_pitch_v} ${imu_yaw_v}"/>
   </joint>
+  <!-- ========================================================= -->
+  <!-- Front caster wheels (passive, fixed in URDF)             -->
+  <!-- ========================================================= -->
+  <link name="front_left_caster_link">
+    <visual>
+      <origin xyz="0 0 0" rpy="${pi/2} 0 0"/>
+      <geometry>
+        <cylinder radius="${front_caster_radius_v}" length="${front_caster_width_v}"/>
+      </geometry>
+      <material name="black"/>
+    </visual>
+    <collision>
+      <origin xyz="0 0 0" rpy="${pi/2} 0 0"/>
+      <geometry>
+        <cylinder radius="${front_caster_radius_v}" length="${front_caster_width_v}"/>
+      </geometry>
+    </collision>
+  </link>
+  <joint name="front_left_caster_joint" type="fixed">
+    <parent link="base_link"/>
+    <child link="front_left_caster_link"/>
+    <origin xyz="${front_caster_x_v} ${front_caster_y_v} ${front_caster_z_v}" rpy="0 0 0"/>
+  </joint>
+  <link name="front_right_caster_link">
+    <visual>
+      <origin xyz="0 0 0" rpy="${pi/2} 0 0"/>
+      <geometry>
+        <cylinder radius="${front_caster_radius_v}" length="${front_caster_width_v}"/>
+      </geometry>
+      <material name="black"/>
+    </visual>
+    <collision>
+      <origin xyz="0 0 0" rpy="${pi/2} 0 0"/>
+      <geometry>
+        <cylinder radius="${front_caster_radius_v}" length="${front_caster_width_v}"/>
+      </geometry>
+    </collision>
+  </link>
+  <joint name="front_right_caster_joint" type="fixed">
+    <parent link="base_link"/>
+    <child link="front_right_caster_link"/>
+    <origin xyz="${front_caster_x_v} ${-front_caster_y_v} ${front_caster_z_v}" rpy="0 0 0"/>
+  </joint>
 </robot>

Commit message: PID, encoder sign match, lidar frame match, imu topic sign match odom topic sign match

File: ros2_ws/src/wheelchair_description/urdf/wheelchair.urdf.xacro (robot description, xacro)
@@ -89,5 +89,5 @@
   <!-- LiDAR                                                     -->
   <!-- ========================================================= -->
-  <link name="lidar_link">
+  <link name="ldlidar_base">
     <visual>
       <origin xyz="0 0 0" rpy="0 0 0"/>
@@ -100,5 +100,5 @@
   <joint name="lidar_joint" type="fixed">
     <parent link="base_link"/>
-    <child link="lidar_link"/>
+    <child link="ldlidar_base"/>
     <origin xyz="${lidar_x_v} ${lidar_y_v} ${lidar_z_v}"
             rpy="${lidar_roll_v} ${lidar_pitch_v} ${lidar_yaw_v}"/>

Commit message: edited URDF, RPP configuration. Implemented MPPI version of self-driving

File: ros2_ws/src/wheelchair_description/urdf/wheelchair.urdf.xacro (robot description, xacro)
@@ -5,11 +5,11 @@
   <!-- ========================================================= -->
   <!-- Base body -->
-  <xacro:arg name="base_length" default="0.650"/>
-  <xacro:arg name="base_width"  default="0.447"/>
+  <xacro:arg name="base_length" default="0.820"/>
+  <xacro:arg name="base_width"  default="0.640"/>
   <xacro:arg name="base_height" default="0.260"/>
   <xacro:arg name="base_z"      default="0.171"/>
   <!-- LiDAR mount -->
-  <xacro:arg name="lidar_x" default="0.680"/>
-  <xacro:arg name="lidar_y" default="0.2175"/>
+  <xacro:arg name="lidar_x" default="0.500"/>
+  <xacro:arg name="lidar_y" default="0.210"/>
   <xacro:arg name="lidar_z" default="0.471"/>
   <xacro:arg name="lidar_roll"  default="0.0"/>
@@ -17,13 +17,13 @@
   <xacro:arg name="lidar_yaw"   default="0.0"/>
   <!-- IMU mount -->
-  <xacro:arg name="imu_x" default="0.325"/>
-  <xacro:arg name="imu_y" default="0.0"/>
+  <xacro:arg name="imu_x" default="0.03"/>
+  <xacro:arg name="imu_y" default="0.015"/>
   <xacro:arg name="imu_z" default="0.342"/>
   <xacro:arg name="imu_roll"  default="0.0"/>
   <xacro:arg name="imu_pitch" default="0.0"/>
-  <xacro:arg name="imu_yaw"   default="0.0"/>
+  <xacro:arg name="imu_yaw"   default="6.28"/>
   <!-- Front caster wheels -->
-  <xacro:arg name="front_caster_x"      default="0.650"/>
-  <xacro:arg name="front_caster_y"      default="0.2235"/>
+  <xacro:arg name="front_caster_x"      default="0.450"/>
+  <xacro:arg name="front_caster_y"      default="0.210"/>
   <xacro:arg name="front_caster_z"      default="-0.079"/>
   <xacro:arg name="front_caster_radius" default="0.092"/>
@@ -68,5 +68,5 @@
   <link name="base_link">
     <visual>
-      <origin xyz="0 0 ${float(base_height_v)/2.0}" rpy="0 0 0"/>
+      <origin xyz="0.110 0 ${float(base_height_v)/2.0}" rpy="0 0 0"/>
       <geometry>
         <box size="${base_length_v} ${base_width_v} ${base_height_v}"/>
@@ -75,5 +75,5 @@
     </visual>
     <collision>
-      <origin xyz="0 0 ${float(base_height_v)/2.0}" rpy="0 0 0"/>
+      <origin xyz="0.110 0 ${float(base_height_v)/2.0}" rpy="0 0 0"/>
       <geometry>
         <box size="${base_length_v} ${base_width_v} ${base_height_v}"/>
